Commit message: Remake of seven DOF arm

File: demo_robot_description_pkg/urdf/sensors/xtion_pro_live.urdf.xacro (robot description, xacro)
@@ -27,10 +27,17 @@
       </inertial>
       <visual>
-        <origin xyz="0 0 0" rpy="0 0 0"/>
-        <geometry>
-          <mesh filename="package://demo_robot_description_pkg/meshes/sensors/xtion_pro_live/xtion_pro_live.dae"/>
+         <geometry>
+          <!--
+          <box size="0.06 0.1 0.03" />
+        	-->
+					<mesh filename="package://mastering_ros_robot_description_pkg/meshes/sensors/xtion_pro_live/xtion_pro_live.stl"/>
         </geometry>
         <material name="DarkGrey"/>
       </visual>
+      <collision>
+      <geometry>
+          <mesh filename="package://mastering_ros_robot_description_pkg/meshes/sensors/xtion_pro_live/xtion_pro_live.dae"/>
+      </geometry>
+      </collision>
     </link>
     <joint name="${name}_optical_joint" type="fixed">

Commit message: Changed mesh file source package

File: demo_robot_description_pkg/urdf/sensors/xtion_pro_live.urdf.xacro (robot description, xacro)
@@ -31,5 +31,5 @@
           <box size="0.06 0.1 0.03" />
         	-->
-					<mesh filename="package://mastering_ros_robot_description_pkg/meshes/sensors/xtion_pro_live/xtion_pro_live.stl"/>
+					<mesh filename="package://demo_robot_description_pkg/meshes/sensors/xtion_pro_live/xtion_pro_live.stl"/>
         </geometry>
         <material name="DarkGrey"/>
@@ -37,5 +37,5 @@
       <collision>
       <geometry>
-          <mesh filename="package://mastering_ros_robot_description_pkg/meshes/sensors/xtion_pro_live/xtion_pro_live.dae"/>
+          <mesh filename="package://demo_robot_description_pkg/meshes/sensors/xtion_pro_live/xtion_pro_live.dae"/>
       </geometry>
       </collision>
