Commit message: Updated with 3rd edition repo copies

File: demo_robot_description_pkg/urdf/diff_wheeled_robot.xacro (robot description, xacro)
@@ -1,6 +1,6 @@
 <?xml version="1.0"?>
-<robot name="diff_wheeled_robot" xmlns:xacro="http://ros.org/wiki/xacro">
-<xacro:include filename="$(find demo_robot_description_pkg)/urdf/wheel.urdf.xacro" />
-<!-- Colours -->
+<robot name="differential_wheeled_robot" xmlns:xacro="http://ros.org/wiki/xacro">
+  <xacro:include filename="$(find demo_robot_description_pkg)/urdf/wheel.urdf.xacro" />
+<!-- Defining the colors used in this robot -->
   <material name="Black">
     <color rgba="0.0 0.0 0.0 1.0"/>
@@ -24,10 +24,10 @@
   <xacro:property name="base_height" value="0.02" />
   <xacro:property name="base_radius" value="0.15" />
-  <xacro:property name="base_mass" value="5" /> <!-- in kg-->
+  <xacro:property name="base_mass" value="5.0" /> <!-- in kg-->
   <!-- caster wheel radius and height -->
   <!-- caster wheel mass -->
   <xacro:property name="caster_f_height" value="0.04" />
   <xacro:property name="caster_f_radius" value="0.025" />
-  <xacro:property name="caster_f_mass" value="0.5" /> <!-- in kg-->
+  <xacro:property name="caster_f_mass" value="0.5" />
   <!-- caster wheel radius and height -->
   <!-- caster wheel mass -->
@@ -66,127 +66,122 @@
   </link>
   <gazebo reference="base_footprint">
-        <turnGravityOff>false</turnGravityOff>
+    <turnGravityOff>false</turnGravityOff>
   </gazebo>
   <joint name="base_footprint_joint" type="fixed">
-        <origin xyz="0 0 ${wheel_radius - base_z_origin_to_wheel_origin}" rpy="0 0 0" />
-        <parent link="base_footprint"/>
-        <child link="base_link" />
+    <origin xyz="0 0 ${wheel_radius - base_z_origin_to_wheel_origin}" rpy="0 0 0" />
+    <parent link="base_footprint"/>
+    <child link="base_link" />
   </joint>
-  <!-- BASE-LINK -->
-  <!--Actual body/chassis of the robot-->
   <link name="base_link">
     <inertial>
-        <mass value="5" />
-        <origin xyz="0 0 0" />
-        <inertia ixx="0.0001" ixy="0.0" ixz="0.0"
+      <mass value="${base_mass}" />
+      <origin xyz="0 0 0" />
+      <inertia ixx="0.0001" ixy="0.0" ixz="0.0"
           iyy="0.0001" iyz="0.0"
           izz="0.0001" />
+      <cylinder_inertia  m="${base_mass}" r="${base_radius}" h="${base_height}" />
     </inertial>
     <visual>
-        <origin xyz="0 0 0" rpy="0 0 0" />
-        <geometry>
-            <cylinder length="0.015" radius="0.10" />
-        </geometry>
-        <material name="White" />
+      <origin xyz="0 0 0" rpy="0 0 0" />
+      <geometry>
+          <cylinder length="${base_height}" radius="${base_radius}" />
+      </geometry>
+      <material name="White" />
     </visual>
     <collision>
-        <origin xyz="0 0 0" rpy="0 0 0 " />
-        <geometry>
-            <cylinder length=".02" radius="0.15" />
-        </geometry>
+      <origin xyz="0 0 0" rpy="0 0 0 " />
+      <geometry>
+          <cylinder length="${base_height}" radius="${base_radius}" />
+      </geometry>
     </collision>
   </link>
   <gazebo reference="base_link">
-        <material>Gazebo/White</material>
-        <turnGravityOff>false</turnGravityOff>
+    <material>Gazebo/White</material>
+    <turnGravityOff>false</turnGravityOff>
   </gazebo>
-<!--Caster front  -->
-    <link name="caster_front_link">
-        <visual>
-            <origin xyz="0 0.02 0" rpy="${M_PI/2} 0 0" />
-            <geometry>
-                <sphere radius="${caster_f_radius}" />
-            </geometry>
-            <material name="Black" />
-        </visual>
-        <collision>
-            <geometry>
-                <sphere radius="${caster_f_radius}" />
-            </geometry>
-            <origin xyz="0 0.02 0" rpy="${M_PI/2} 0 0" />
-        </collision>
-        <inertial>
-            <mass value="${caster_f_mass}" />
-            <origin xyz="0 0 0" />
-            <inertia ixx="0.001" ixy="0.0" ixz="0.0"
-                    iyy="0.001" iyz="0.0"
-                    izz="0.001" />
-            </inertial>
-    </link>
-    <joint name="caster_front_joint" type="fixed">
-        <parent link="base_link"/>
-        <child link="caster_front_link"/>
-        <origin xyz="0.115 0.0 0.007" rpy="${-M_PI/2} 0 0"/>
-    </joint>
-    <gazebo reference="caster_front_link">
-        <turnGravityOff>false</turnGravityOff>
-    </gazebo>
-<!--Caster back  -->
-    <link name="caster_back_link">
+  <link name="caster_front_link">
     <visual>
-        <origin xyz="0.02 0.02 0 " rpy="${M_PI/2} 0 0" />
-        <geometry>
-            <sphere radius="${caster_b_radius}" />
-        </geometry>
-        <material name="Black" />
+      <origin xyz="0 0.02 0" rpy="${M_PI/2} 0 0" />
+      <geometry>
+				<sphere radius="${caster_f_radius}" />
+      </geometry>
+      <material name="Black" />
     </visual>
     <collision>
-        <geometry>
-		    <sphere radius="${caster_b_radius}" />
-        </geometry>
-        <origin xyz="0 0.02 0 " rpy="${M_PI/2} 0 0" />
+      <geometry>
+				<sphere radius="${caster_f_radius}" />
+      </geometry>
+    <origin xyz="0 0.02 0" rpy="${M_PI/2} 0 0" />
     </collision>
     <inertial>
-        <mass value="${caster_b_mass}" />
-        <origin xyz="0 0 0" />
-        <inertia ixx="0.001" ixy="0.0" ixz="0.0"
-                iyy="0.001" iyz="0.0"
-                izz="0.001" />
+      <mass value="${caster_f_mass}" />
+      <origin xyz="0 0 0" />
+      <inertia ixx="0.001" ixy="0.0" ixz="0.0"
+               iyy="0.001" iyz="0.0"
+               izz="0.001" />
     </inertial>
-    </link>
-    <joint name="caster_back_joint" type="fixed">
-        <parent link="base_link"/>
-        <child link="caster_back_link"/>
-        <origin xyz="-0.135 0.0 0.009" rpy="${-M_PI/2} 0 0"/>
-    </joint>
-    <gazebo reference="caster_back_link">
-        <turnGravityOff>false</turnGravityOff>
-    </gazebo>
-    <!-- Wheel Definitions -->
-    <wheel fb="front" lr="right" parent="base_link" translateX="0" translateY="0.5" flipY="1"/>
-    <wheel fb="front" lr="left" parent="base_link" translateX="0" translateY="-0.5" flipY="1"/>
-    <!-- Differential drive controller  -->
-    <gazebo>
-        <plugin name="differential_drive_controller" filename="libgazebo_ros_diff_drive.so">
-            <legacyMode>true</legacyMode>
-            <rosDebugLevel>Debug</rosDebugLevel>
-            <publishWheelTF>false</publishWheelTF>
-            <robotNamespace>/</robotNamespace>
-            <publishTf>1</publishTf>
-            <publishWheelJointState>false</publishWheelJointState>
-            <alwaysOn>true</alwaysOn>
-            <updateRate>100.0</updateRate>
-            <leftJoint>front_left_wheel_joint</leftJoint>
-            <rightJoint>front_right_wheel_joint</rightJoint>
-            <wheelSeparation>${2*base_radius}</wheelSeparation>
-            <wheelDiameter>${2*wheel_radius}</wheelDiameter>
-            <broadcastTF>1</broadcastTF>
-            <wheelTorque>30</wheelTorque>
-            <wheelAcceleration>1.8</wheelAcceleration>
-            <commandTopic>cmd_vel</commandTopic>
-            <odometryFrame>odom</odometryFrame>
-            <odometryTopic>odom</odometryTopic>
-            <robotBaseFrame>base_footprint</robotBaseFrame>
-        </plugin>
-    </gazebo>
+  </link>
+	<joint name="caster_front_joint" type="fixed">
+    <parent link="base_link"/>
+    <child link="caster_front_link"/>
+    <origin xyz="0.115 0.0 0.007" rpy="${-M_PI/2} 0 0"/>
+  </joint>
+  <gazebo reference="caster_front_link">
+    <turnGravityOff>false</turnGravityOff>
+  </gazebo>
+  <link name="caster_back_link">
+  <visual>
+    <origin xyz="0.02 0.02 0 " rpy="${M_PI/2} 0 0" />
+    <geometry>
+			<sphere radius="${caster_b_radius}" />
+    </geometry>
+    <material name="Black" />
+  </visual>
+  <collision>
+    <geometry>
+			<sphere radius="${caster_b_radius}" />
+     </geometry>
+     <origin xyz="0 0.02 0 " rpy="${M_PI/2} 0 0" />
+    </collision>
+    <inertial>
+      <mass value="${caster_b_mass}" />
+      <origin xyz="0 0 0" />
+      <inertia ixx="0.001" ixy="0.0" ixz="0.0"
+               iyy="0.001" iyz="0.0"
+               izz="0.001" />
+    </inertial>
+  </link>
+  <joint name="caster_back_joint" type="fixed">
+    <parent link="base_link"/>
+    <child link="caster_back_link"/>
+    <origin xyz="-0.135 0.0 0.009" rpy="${-M_PI/2} 0 0"/>
+  </joint>
+  <gazebo reference="caster_back_link">
+   <turnGravityOff>false</turnGravityOff>
+  </gazebo>
+  <xacro:wheel fb="front" lr="right" parent="base_link" translateX="0" translateY="-0.5" flipY="1"/>
+	<xacro:wheel fb="front" lr="left" parent="base_link" translateX="0" translateY="0.5" flipY="1"/>
+	<gazebo>
+  	<plugin name="differential_drive_controller" filename="libgazebo_ros_diff_drive.so">
+	    <legacyMode>true</legacyMode>
+	    <rosDebugLevel>Debug</rosDebugLevel>
+	    <publishWheelTF>false</publishWheelTF>
+	    <robotNamespace>/</robotNamespace>
+	    <publishTf>1</publishTf>
+	    <publishWheelJointState>false</publishWheelJointState>
+	    <alwaysOn>true</alwaysOn>
+	    <updateRate>100.0</updateRate>
+	    <leftJoint>front_left_wheel_joint</leftJoint>
+	    <rightJoint>front_right_wheel_joint</rightJoint>
+	    <wheelSeparation>${2*base_radius}</wheelSeparation>
+	    <wheelDiameter>${2*wheel_radius}</wheelDiameter>
+	    <broadcastTF>1</broadcastTF>
+	    <wheelTorque>30</wheelTorque>
+	    <wheelAcceleration>1.8</wheelAcceleration>
+	    <commandTopic>cmd_vel</commandTopic>
+	    <odometryFrame>odom</odometryFrame>
+	    <odometryTopic>odom</odometryTopic>
+	    <robotBaseFrame>base_footprint</robotBaseFrame>
+   </plugin>
+  </gazebo>
 </robot>

File: demo_robot_description_pkg/urdf/wheel.urdf.xacro (robot description, xacro)
@@ -8,55 +8,52 @@
   <xacro:property name="base_y_origin_to_wheel_origin" value="0.3" />
   <xacro:property name="base_z_origin_to_wheel_origin" value="0.0" />
-  <xacro:macro name="cylinder_inertia" params="m r h">
-        <inertia  ixx="${m*(3*r*r+h*h)/12}" ixy = "0" ixz = "0"
-                iyy="${m*(3*r*r+h*h)/12}" iyz = "0"
-                izz="${m*r*r/2}" />
-  </xacro:macro>
   <xacro:macro name="wheel" params="fb lr parent translateX translateY flipY"> <!--fb : front, back ; lr: left, right -->
     <link name="${fb}_${lr}_wheel">
-        <visual>
-            <origin xyz="0 0 0" rpy="${flipY*M_PI/2} 0  0 " />
-            <geometry>
-            <cylinder length="${wheel_height}" radius="${wheel_radius}" />
-            </geometry>
-            <material name="DarkGray" />
-        </visual>
-        <collision>
-            <origin xyz="0 0 0" rpy="${flipY*M_PI/2} 0 0 " />
-            <geometry>
-            <cylinder length="${wheel_height}" radius="${wheel_radius}" />
-            </geometry>
-        </collision>
-        <inertial>
-            <mass value="${wheel_mass}" />
-            <origin xyz="0 0 0" />
-            <cylinder_inertia  m="${wheel_mass}" r="${wheel_radius}" h="${wheel_height}" />
-        </inertial>
+      <visual>
+        <origin xyz="0 0 0" rpy="${flipY*M_PI/2} 0  0 " />
+        <geometry>
+          <cylinder length="${wheel_height}" radius="${wheel_radius}" />
+        </geometry>
+        <material name="DarkGray" />
+      </visual>
+      <collision>
+        <origin xyz="0 0 0" rpy="${flipY*M_PI/2} 0 0 " />
+        <geometry>
+          <cylinder length="${wheel_height}" radius="${wheel_radius}" />
+        </geometry>
+      </collision>
+      <inertial>
+        <mass value="${wheel_mass}" />
+        <origin xyz="0 0 0" />
+				<inertia ixx="0.001" ixy="0.0" ixz="0.0"
+               iyy="0.001" iyz="0.0"
+               izz="0.001" />
+      </inertial>
     </link>
     <gazebo reference="${fb}_${lr}_wheel">
-        <mu1 value="1.0"/>
-        <mu2 value="1.0"/>
-        <kp  value="10000000.0" />
-        <kd  value="1.0" />
-        <fdir1 value="1 0 0"/>
-        <material>Gazebo/Grey</material>
-        <turnGravityOff>false</turnGravityOff>
+      <mu1 value="1.0"/>
+      <mu2 value="1.0"/>
+      <kp  value="10000000.0" />
+      <kd  value="1.0" />
+      <fdir1 value="1 0 0"/>
+      <material>Gazebo/Grey</material>
+      <turnGravityOff>false</turnGravityOff>
     </gazebo>
     <joint name="${fb}_${lr}_wheel_joint" type="continuous">
-        <parent link="${parent}"/>
-        <child link="${fb}_${lr}_wheel"/>
-        <origin xyz="${translateX * base_x_origin_to_wheel_origin} ${translateY * base_y_origin_to_wheel_origin} ${base_z_origin_to_wheel_origin}" rpy="0 0 0" />
-        <axis xyz="0 1 0" rpy="0  0" />
-        <limit effort="100" velocity="100"/>
-        <joint_properties damping="0.0" friction="0.0"/>
+      <parent link="${parent}"/>
+      <child link="${fb}_${lr}_wheel"/>
+      <origin xyz="${translateX * base_x_origin_to_wheel_origin} ${translateY * base_y_origin_to_wheel_origin} ${base_z_origin_to_wheel_origin}" rpy="0 0 0" />
+      <axis xyz="0 1 0" rpy="0 0 0" />
+      <limit effort="100" velocity="100"/>
+      <joint_properties damping="0.0" friction="0.0"/>
     </joint>
     <!-- Transmission is important to link the joints and the controller -->
     <transmission name="${fb}_${lr}_wheel_joint_trans">
-        <type>transmission_interface/SimpleTransmission</type>
-        <joint name="${fb}_${lr}_wheel_joint" />
-        <actuator name="${fb}_${lr}_wheel_joint_motor">
-            <hardwareInterface>EffortJointInterface</hardwareInterface>
-            <mechanicalReduction>1</mechanicalReduction>
-        </actuator>
+      <type>transmission_interface/SimpleTransmission</type>
+      <joint name="${fb}_${lr}_wheel_joint" />
+      <actuator name="${fb}_${lr}_wheel_joint_motor">
+        <hardwareInterface>EffortJointInterface</hardwareInterface>
+        <mechanicalReduction>1</mechanicalReduction>
+      </actuator>
     </transmission>
   </xacro:macro>

Commit message: Added RVIZ Pan_tilt config

File: demo_robot_description_pkg/urdf/diff_wheeled_robot.xacro (robot description, xacro)
@@ -160,6 +160,43 @@
    <turnGravityOff>false</turnGravityOff>
   </gazebo>
+  <!-- Laser Joint -->
+  <joint name="hokuyo_joint" type="fixed">
+    <origin xyz="${base_radius - hokuyo_size/2} 0 ${base_height+hokuyo_size/4}" rpy="0 0 0" />
+    <parent link="base_link"/>
+    <child link="laser_link" />
+  </joint>
+  <!-- Gazebo Laser Plugin Setup -->
+  <gazebo reference="laser_link">
+    <material>Gazebo/Blue</material>
+    <turnGravityOff>false</turnGravityOff>
+    <sensor type="ray" name="head_hokuyo_sensor">
+      <pose>${hokuyo_size/2} 0 0 0 0 0</pose>
+      <visualize>true</visualize>
+      <update_rate>40</update_rate>
+      <ray>
+        <scan>
+          <horizontal>
+            <samples>720</samples>
+            <resolution>1</resolution>
+            <min_angle>-1.570796</min_angle>
+            <max_angle>1.570796</max_angle>
+          </horizontal>
+        </scan>
+        <range>
+          <min>0.10</min>
+          <max>10.0</max>
+          <resolution>0.001</resolution>
+        </range>
+      </ray>
+      <plugin name="gazebo_ros_head_hokuyo_controller" filename="libgazebo_ros_laser.so">
+        <topicName>/scan</topicName>
+        <frameName>laser_link</frameName>
+      </plugin>
+    </sensor>
+  </gazebo>
+  <!-- Wheels -->
   <xacro:wheel fb="front" lr="right" parent="base_link" translateX="0" translateY="-0.5" flipY="1"/>
 	<xacro:wheel fb="front" lr="left" parent="base_link" translateX="0" translateY="0.5" flipY="1"/>
+  <!-- Gazebo Differential Drive Controller Setup -->
 	<gazebo>
   	<plugin name="differential_drive_controller" filename="libgazebo_ros_diff_drive.so">

Commit message: added dark grey material

File: demo_robot_description_pkg/urdf/diff_wheeled_robot.xacro (robot description, xacro)
@@ -11,4 +11,7 @@
   <material name="White">
     <color rgba="1.0 1.0 1.0 1.0"/>
+  </material>
+  <material name="DarkGray">
+    <color rgba="0.7 0.7 0.7 1.0"/>
   </material>
   <material name="Blue">
@@ -161,11 +164,11 @@
   </gazebo>
   <!-- Laser Joint -->
-  <joint name="hokuyo_joint" type="fixed">
+  <!-- <joint name="hokuyo_joint" type="fixed">
     <origin xyz="${base_radius - hokuyo_size/2} 0 ${base_height+hokuyo_size/4}" rpy="0 0 0" />
     <parent link="base_link"/>
     <child link="laser_link" />
-  </joint>
+  </joint> -->
   <!-- Gazebo Laser Plugin Setup -->
-  <gazebo reference="laser_link">
+  <!-- <gazebo reference="laser_link">
     <material>Gazebo/Blue</material>
     <turnGravityOff>false</turnGravityOff>
@@ -194,5 +197,5 @@
       </plugin>
     </sensor>
-  </gazebo>
+  </gazebo> -->
   <!-- Wheels -->
   <xacro:wheel fb="front" lr="right" parent="base_link" translateX="0" translateY="-0.5" flipY="1"/>
